Commit message: Parametrize delta urdfs, separate namespace.

File: rotors_description/urdf/delta_actuators.xacro (robot description, xacro)
@@ -1,4 +1,4 @@
 <?xml version="1.0"?>
-<robot name="$(arg mav_name)" xmlns:xacro="http://ros.org/wiki/xacro">
+<robot name="${robot_name}" xmlns:xacro="http://ros.org/wiki/xacro">
   <!-- Relationship between the p, d gain and the closed-loop dynamics behaviour of the system:
   It behaves like a second-order system in the frequency domain: Y(s) = U(s)*(ds + p)/(Is**2 + ds + p)
@@ -7,8 +7,14 @@
    -->
 <xacro:property name="delta_control_mode" value="$(arg delta_control_mode)" />
+<xacro:property name="servo_zero_offset" value="0.0" />
+<!-- cmd_min/max = 0 for unlimited -->
+<xacro:property name="servo_cmd_min" value="-100.0" />
+<xacro:property name="servo_cmd_max" value="100.0" />
+<xacro:property name="servo_i_min" value="-20.0" />
+<xacro:property name="servo_i_max" value="20.0" />
 <xacro:if value="${delta_control_mode == 'position'}">
-  <xacro:property name="p_gain_delta" value="0.5" />
-  <xacro:property name="i_gain_delta" value="0.01" />
-  <xacro:property name="d_gain_delta" value="0.1" />
+  <xacro:property name="p_gain_delta" value="5.0" />
+  <xacro:property name="i_gain_delta" value="0.1" />
+  <xacro:property name="d_gain_delta" value="1.0" />
 </xacro:if>
 <xacro:if value="${delta_control_mode == 'velocity'}">
@@ -25,9 +31,9 @@
   <!-- Add motors. -->
   <gazebo>
-      <plugin name="multimotor_plugin" filename="librotors_gazebo_multimotor_plugin.so">
-        <robotNamespace>$(arg mav_name)</robotNamespace>
+      <plugin name="delta_multimotor_plugin" filename="librotors_gazebo_multimotor_plugin.so">
+        <robotNamespace>${delta_namespace}</robotNamespace>
         <servos>
             <servo>
-              <jointName>${namespace}/delta_joint_upper_0</jointName>
+              <jointName>${delta_namespace}/delta_joint_upper_0</jointName>
               <spinDirection>cw</spinDirection>
               <controlMode>${delta_control_mode}</controlMode>
@@ -35,17 +41,17 @@
               <minRotPosition>${-pi}</minRotPosition>
               <maxRotPosition>${pi}</maxRotPosition>
-              <zeroOffset>0.0</zeroOffset>
+              <zeroOffset>${servo_zero_offset}</zeroOffset>
               <joint_control_pid>
                   <p>${p_gain_delta}</p>
                   <i>${i_gain_delta}</i>
                   <d>${d_gain_delta}</d>
-                  <iMax>1.0</iMax>
-                  <iMin>-1.0</iMin>
-                  <cmdMax>2.0</cmdMax>
-                  <cmdMin>-2.0</cmdMin>
+                  <iMax>${servo_i_max}</iMax>
+                  <iMin>${servo_i_min}</iMin>
+                  <cmdMax>${servo_cmd_max}</cmdMax>
+                  <cmdMin>${servo_cmd_min}</cmdMin>
               </joint_control_pid>
             </servo>
             <servo>
-              <jointName>${namespace}/delta_joint_upper_1</jointName>
+              <jointName>${delta_namespace}/delta_joint_upper_1</jointName>
               <spinDirection>cw</spinDirection>
               <controlMode>${delta_control_mode}</controlMode>
@@ -53,17 +59,17 @@
               <minRotPosition>${-pi}</minRotPosition>
               <maxRotPosition>${pi}</maxRotPosition>
-              <zeroOffset>0.0</zeroOffset>
+              <zeroOffset>${servo_zero_offset}</zeroOffset>
               <joint_control_pid>
                   <p>${p_gain_delta}</p>
                   <i>${i_gain_delta}</i>
                   <d>${d_gain_delta}</d>
-                  <iMax>1.0</iMax>
-                  <iMin>-1.0</iMin>
-                  <cmdMax>2.0</cmdMax>
-                  <cmdMin>-2.0</cmdMin>
+                  <iMax>${servo_i_max}</iMax>
+                  <iMin>${servo_i_min}</iMin>
+                  <cmdMax>${servo_cmd_max}</cmdMax>
+                  <cmdMin>${servo_cmd_min}</cmdMin>
               </joint_control_pid>
             </servo>
             <servo>
-              <jointName>${namespace}/delta_joint_upper_2</jointName>
+              <jointName>${delta_namespace}/delta_joint_upper_2</jointName>
               <spinDirection>cw</spinDirection>
               <controlMode>${delta_control_mode}</controlMode>
@@ -71,13 +77,13 @@
               <minRotPosition>${-pi}</minRotPosition>
               <maxRotPosition>${pi}</maxRotPosition>
-              <zeroOffset>0.0</zeroOffset>
+              <zeroOffset>${servo_zero_offset}</zeroOffset>
               <joint_control_pid>
                   <p>${p_gain_delta}</p>
                   <i>${i_gain_delta}</i>
                   <d>${d_gain_delta}</d>
-                  <iMax>1.0</iMax>
-                  <iMin>-1.0</iMin>
-                  <cmdMax>2.0</cmdMax>
-                  <cmdMin>-2.0</cmdMin>
+                  <iMax>${servo_i_max}</iMax>
+                  <iMin>${servo_i_min}</iMin>
+                  <cmdMax>${servo_cmd_max}</cmdMax>
+                  <cmdMin>${servo_cmd_min}</cmdMin>
               </joint_control_pid>
             </servo>

File: rotors_description/urdf/delta_base.xacro (robot description, xacro)
@@ -48,5 +48,5 @@
   </link>
   <xacro:property name="robot_name" value="$(arg mav_name)" />
-  <xacro:property name="namespace" value="$(arg namespace)" />
+  <xacro:property name="delta_namespace" value="$(arg namespace)" />
   <xacro:property name="mounting_link" value="${namespace}/base_link" />
   <xacro:property name="height_offset" value="0.0" />

File: rotors_description/urdf/delta_elements.xacro (robot description, xacro)
@@ -129,5 +129,5 @@
     <!-- Base Plate Link Macro -->
     <xacro:macro name="base_plate_macro">
-        <link name="${namespace}/delta_base_link">
+        <link name="${delta_namespace}/delta_base_link">
 <!--             <visual>
                 <xacro:insert_block name="base_plate_origin"/>
@@ -146,5 +146,5 @@
     <!-- Proximal Link Macro -->
     <xacro:macro name="link1_macro" params="suffix">
-        <link name="${namespace}/delta_link1_${suffix}">
+        <link name="${delta_namespace}/delta_link1_${suffix}">
             <visual>
                 <xacro:insert_block name="link_proximal_origin"/>
@@ -164,5 +164,5 @@
     <xacro:macro name="link2_right_macro" params="suffix base_angle">
         <gazebo>
-            <link name="${namespace}/delta_link2_right_${suffix}">
+            <link name="${delta_namespace}/delta_link2_right_${suffix}">
                 <pose>
                 ${(tool_plate_radius-link_distal_length*sin(angle_offset))*cos(base_angle)+(link_proximal_width/2)*sin(base_angle)}
@@ -186,5 +186,5 @@
     <xacro:macro name="link2_left_macro" params="suffix base_angle">
         <gazebo>
-            <link name="${namespace}/delta_link2_left_${suffix}">
+            <link name="${delta_namespace}/delta_link2_left_${suffix}">
                 <pose>
                 ${(tool_plate_radius-link_distal_length*sin(angle_offset))*cos(base_angle)+(-link_proximal_width/2)*sin(base_angle)}
@@ -209,5 +209,5 @@
     <xacro:macro name="tool_plate_macro">
         <gazebo>
-            <link name='${namespace}/delta_tool_plate'>
+            <link name='${delta_namespace}/delta_tool_plate'>
                 <pose>${tool_plate_radius}
                     ${-link_proximal_width/2}
@@ -235,7 +235,7 @@
     -->
     <xacro:macro name="shoulder_joint_macro" params="suffix base_angle motor_start_index">
-        <joint name="${namespace}/delta_joint_upper_${suffix}" type="continuous">
-            <parent link="${namespace}/delta_base_link"/>
-            <child link="${namespace}/delta_link1_${suffix}"/>
+        <joint name="${delta_namespace}/delta_joint_upper_${suffix}" type="continuous">
+            <parent link="${delta_namespace}/delta_base_link"/>
+            <child link="${delta_namespace}/delta_link1_${suffix}"/>
             <origin xyz="${base_plate_radius*cos(base_angle)} ${base_plate_radius*sin(base_angle)} 0.0" rpy="0.0 0.0 ${base_angle}"/>
             <axis xyz="0.0 1.0 0.0"/>
@@ -246,7 +246,7 @@
 <!--         <gazebo>
           <plugin name="delta_${suffix}_motor_model" filename="librotors_gazebo_motor_model.so">
-            <robotNamespace>${namespace}</robotNamespace>
-            <jointName>${namespace}/delta_joint_upper_${suffix}</jointName>
-            <linkName>${namespace}/delta_link1_${suffix}</linkName>
+            <robotNamespace>${delta_namespace}</robotNamespace>
+            <jointName>${delta_namespace}/delta_joint_upper_${suffix}</jointName>
+            <linkName>${delta_namespace}/delta_link1_${suffix}</linkName>
             <turningDirection>ccw</turningDirection>
             <motorType>position</motorType>
@@ -269,7 +269,7 @@
     <xacro:macro name="universal_middle_joint_macro" params="type suffix base_angle">
         <gazebo>
-            <joint name='${namespace}/delta_joint_middle_${type}_${suffix}' type='universal'>
-                <child>${namespace}/delta_link2_${type}_${suffix}</child>
-                <parent>${namespace}/delta_link1_${suffix}</parent>
+            <joint name='${delta_namespace}/delta_joint_middle_${type}_${suffix}' type='universal'>
+                <child>${delta_namespace}/delta_link2_${type}_${suffix}</child>
+                <parent>${delta_namespace}/delta_link1_${suffix}</parent>
                 <axis>
                     <xyz>${-sin(base_angle)} ${cos(base_angle)} 0</xyz>
@@ -291,7 +291,7 @@
     <xacro:macro name="universal_lower_joint_macro" params="type suffix base_angle">
         <gazebo>
-            <joint name='${namespace}/delta_joint_lower_${type}_${suffix}' type='universal'>
-                <child>${namespace}/delta_link2_${type}_${suffix}</child>
-                <parent>${namespace}/delta_tool_plate</parent>
+            <joint name='${delta_namespace}/delta_joint_lower_${type}_${suffix}' type='universal'>
+                <child>${delta_namespace}/delta_link2_${type}_${suffix}</child>
+                <parent>${delta_namespace}/delta_tool_plate</parent>
                 <pose>0 0 ${link_distal_length} 0 0 0</pose>
                 <axis>
@@ -324,5 +324,5 @@
     <gazebo>
     <!-- odometry link -->
-    <link name="${namespace}/odometry_sensor_${odometry_sensor_suffix}_link">
+    <link name="${delta_namespace}/odometry_sensor_${odometry_sensor_suffix}_link">
         <pose>0 0 ${-link_proximal_length*sin(angle_offset)+base_plate_height/2+tool_plate_height/2+height_offset} 0 0 0</pose>
         <inertial>
@@ -340,7 +340,7 @@
     </link>
     <!-- odometry joint -->
-    <joint name="${namespace}/odometry_sensor${odometry_sensor_suffix}_joint" type="revolute">
+    <joint name="${delta_namespace}/odometry_sensor${odometry_sensor_suffix}_joint" type="revolute">
       <parent> ${parent_link} </parent>
-      <child> ${namespace}/odometry_sensor_${odometry_sensor_suffix}_link </child>
+      <child> ${delta_namespace}/odometry_sensor_${odometry_sensor_suffix}_link </child>
       <pose>0 0 0 0 0 0</pose>
       <axis>
@@ -360,6 +360,6 @@
     </joint>
       <plugin filename="librotors_gazebo_odometry_plugin.so" name="odometry_sensor_${odometry_sensor_suffix}">
-        <linkName>${namespace}/odometry_sensor_${odometry_sensor_suffix}_link</linkName>
-        <robotNamespace>${namespace}</robotNamespace>
+        <linkName>${delta_namespace}/odometry_sensor_${odometry_sensor_suffix}_link</linkName>
+        <robotNamespace>${delta_namespace}</robotNamespace>
         <poseTopic>${pose_topic}</poseTopic>
         <poseWithCovarianceTopic>${pose_with_covariance_topic}</poseWithCovarianceTopic>

File: rotors_description/urdf/delta_manipulator.xacro (robot description, xacro)
@@ -5,10 +5,10 @@
     <xacro:property name="mounting_link" default="world" />
     <xacro:property name="height_offset" default="-0.07" />
-    <xacro:property name="namespace" default="$(arg mav_name)" />
+    <xacro:property name="delta_namespace" default="${delta_namespace}" />
     <xacro:property name="delta_start_index" default="12" />
     <joint name="mounting_joint" type="fixed">
         <origin xyz="0 0 ${height_offset}" rpy="0.0 0.0 0.0"/>
         <parent link="${mounting_link}"/>
-        <child link="${namespace}/delta_base_link"/>
+        <child link="${delta_namespace}/delta_base_link"/>
     </joint>
     <xacro:base_plate_macro />
@@ -39,7 +39,7 @@
     <xacro:tool_plate_macro />
     <xacro:odometry_plugin_gz_macro
-        namespace="${namespace}"
+        namespace="${delta_namespace}"
         odometry_sensor_suffix="tool"
-        parent_link="${namespace}/delta_tool_plate"
+        parent_link="${delta_namespace}/delta_tool_plate"
         pose_topic="odometry_sensor_tool/pose"
         pose_with_covariance_topic="odometry_sensor_tool/pose_with_covariance"
@@ -48,5 +48,5 @@
         odometry_topic="odometry_sensor_tool/odometry"
         parent_frame_id="world"
-        child_frame_id="${namespace}/odometry_sensor_tool"
+        child_frame_id="${delta_namespace}/odometry_sensor_tool"
         mass_odometry_sensor="0.00001"
         measurement_divisor="16"
