Commit message: specified Rotor location in spherical coordinates

File: rotors_description/urdf/griffin.xacro (robot description, xacro)
@@ -31,5 +31,6 @@
     <xacro:property name="body_height" value="0.35"/>    <!-- [m] -->
     <xacro:property name="mass_rotor" value="0.0065"/>    <!-- [kg] -->
-    <xacro:property name="arm_length" value="0.300"/>    <!-- [m] -->
+    <xacro:property name="arm_length_front" value="0.600"/>    <!-- [m] -->
+    <xacro:property name="arm_length_back" value="0.4"/>
     <xacro:property name="rotor_offset_top" value="0.060"/>    <!-- [m] -->
     <xacro:property name="radius_rotor" value="0.1143"/>    <!-- [m] -->
@@ -44,6 +45,6 @@
     <xacro:property name="velocity_revolute" value="0.5"/>
     <xacro:property name="tilt_input_scaling" value="31.4159" />
-    <xacro:property name="sin30" value="0.5"/>
-    <xacro:property name="cos30" value="0.866025403784"/>
+    <xacro:property name="cos60" value="0.5"/>
+    <xacro:property name="sin60" value="0.866025403784"/>
     <xacro:property name="rotor_drag_coefficient" value="${8.06428e-05}"/>
     <xacro:property name="rolling_moment_coefficient" value="0.000001"/>
@@ -82,5 +83,5 @@
   <!-- Instantiate rotors -->
   <xacro:double_tilt_unit robot_namespace="${namespace}"
-    suffix="right"
+    suffix="left"
     direction_upper="ccw"
     direction_lower="cw"
@@ -105,10 +106,10 @@
     i_gain="${tilt_i_gain}"
     d_gain="${tilt_d_gain}">
-    <origin xyz="0 ${arm_length} 0" rpy="0 0 0"/>
+    <origin xyz="0 -${arm_length_front*sin60} ${arm_length_front*cos60}" rpy="-1.0471975512 0 0"/>
     <xacro:insert_block name="rotor_inertia" />
   </xacro:double_tilt_unit>
   <xacro:double_tilt_unit
     robot_namespace="${namespace}"
-    suffix="left"
+    suffix="right"
     direction_upper="cw"
     direction_lower="ccw"
@@ -133,5 +134,5 @@
     i_gain="${tilt_i_gain}"
     d_gain="${tilt_d_gain}">
-    <origin xyz="0 ${arm_length} 0" rpy="0 0 1.57079632679"/>
+    <origin xyz="0 ${arm_length_front*sin60} ${arm_length_front*cos60}" rpy="1.0471975512 0 0"/>
     <xacro:insert_block name="rotor_inertia" />
   </xacro:double_tilt_unit>
@@ -161,5 +162,5 @@
     i_gain="${tilt_i_gain}"
     d_gain="${tilt_d_gain}">
-    <origin xyz="${cos30*arm_length} ${sin30*arm_length} 0" rpy="0 0 0.52359877559"/>
+    <origin xyz="0 0 ${arm_length_front}" rpy="0 0 3.14159265359"/>
     <xacro:insert_block name="rotor_inertia" />
   </xacro:double_tilt_unit>
@@ -188,59 +189,5 @@
     i_gain="${tilt_i_gain}"
     d_gain="${tilt_d_gain}">
-    <origin xyz="-${cos30*arm_length} -${sin30*arm_length} 0" rpy="0 0 3.66519142919"/>
-    <xacro:insert_block name="rotor_inertia" />
-  </xacro:double_tilt_unit>
-  <xacro:double_tilt_unit robot_namespace="${namespace}"
-    suffix="front_right"
-    direction_upper="cw"
-    direction_lower="ccw"
-    motor_constant="${motor_constant}"
-    motor_constant_lower="${motor_constant_lower}"
-    moment_constant="${moment_constant}"
-    moment_constant_lower="${moment_constant_lower}"
-    parent="${namespace}/base_link"
-    mass_rotor="${mass_rotor}"
-    mass_tilt_unit="${mass_tilt_unit}"
-    time_constant_up="${time_constant_up}"
-    time_constant_down="${time_constant_down}"
-    max_rot_velocity="${max_rot_velocity}"
-    rotor_offset_top="${rotor_offset_top}"
-    motor_number="4"
-    rotor_drag_coefficient="${rotor_drag_coefficient}"
-    rolling_moment_coefficient="${rolling_moment_coefficient}"
-    mesh="propeller"
-    mesh_tilt_unit="${mesh_file_tilt_unit}"
-    color="Orange"
-    p_gain="${tilt_p_gain}"
-    i_gain="${tilt_i_gain}"
-    d_gain="${tilt_d_gain}">
-    <origin xyz="${cos30*arm_length} -${sin30*arm_length} 0" rpy="0 0 5.75958653158"/>
-    <xacro:insert_block name="rotor_inertia" />
-  </xacro:double_tilt_unit>
-  <xacro:double_tilt_unit robot_namespace="${namespace}"
-    suffix="back_left"
-    direction_upper="ccw"
-    direction_lower="cw"
-    motor_constant="${motor_constant}"
-    motor_constant_lower="${motor_constant_lower}"
-    moment_constant="${moment_constant}"
-    moment_constant_lower="${moment_constant_lower}"
-    parent="${namespace}/base_link"
-    mass_rotor="${mass_rotor}"
-    mass_tilt_unit="${mass_tilt_unit}"
-    time_constant_up="${time_constant_up}"
-    time_constant_down="${time_constant_down}"
-    max_rot_velocity="${max_rot_velocity}"
-    rotor_offset_top="${rotor_offset_top}"
-    motor_number="5"
-    rotor_drag_coefficient="${rotor_drag_coefficient}"
-    rolling_moment_coefficient="${rolling_moment_coefficient}"
-    mesh="propeller"
-    mesh_tilt_unit="${mesh_file_tilt_unit}"
-    color="DarkGrey"
-    p_gain="${tilt_p_gain}"
-    i_gain="${tilt_i_gain}"
-    d_gain="${tilt_d_gain}">
-    <origin xyz="-${cos30*arm_length} ${sin30*arm_length} 0" rpy="0 0 2.61799387799"/>
+    <origin xyz="-${arm_length_back} 0 0" rpy="0 0 3.14159265359"/>
     <xacro:insert_block name="rotor_inertia" />
   </xacro:double_tilt_unit>
@@ -318,36 +265,4 @@
           <joint_control_type>velocity</joint_control_type>
         </channel>
-        <channel name="rotor8">
-          <input_index>8</input_index>
-          <input_offset>0</input_offset>
-          <input_scaling>${max_rot_velocity}</input_scaling>
-          <zero_position_disarmed>0</zero_position_disarmed>
-          <zero_position_armed>100</zero_position_armed>
-          <joint_control_type>velocity</joint_control_type>
-        </channel>
-        <channel name="rotor9">
-          <input_index>9</input_index>
-          <input_offset>0</input_offset>
-          <input_scaling>${max_rot_velocity}</input_scaling>
-          <zero_position_disarmed>0</zero_position_disarmed>
-          <zero_position_armed>100</zero_position_armed>Firefly
-          <joint_control_type>velocity</joint_control_type>
-        </channel>
-        <channel name="rotor10">
-          <input_index>10</input_index>
-          <input_offset>0</input_offset>
-          <input_scaling>${max_rot_velocity}</input_scaling>
-          <zero_position_disarmed>0</zero_position_disarmed>
-          <zero_position_armed>100</zero_position_armed>
-          <joint_control_type>velocity</joint_control_type>
-        </channel>
-        <channel name="rotor11">
-          <input_index>11</input_index>
-          <input_offset>0</input_offset>
-          <input_scaling>${max_rot_velocity}</input_scaling>
-          <zero_position_disarmed>0</zero_position_disarmed>
-          <zero_position_armed>100</zero_position_armed>
-          <joint_control_type>velocity</joint_control_type>
-        </channel>
         <channel name="tilt_unit0">
           <input_index>12</input_index>
@@ -376,20 +291,4 @@
         <channel name="tilt_unit3">
           <input_index>15</input_index>
-          <input_offset>0</input_offset>
-          <input_scaling>${tilt_input_scaling}</input_scaling>
-          <zero_position_disarmed>0</zero_position_disarmed>
-          <zero_position_armed>0</zero_position_armed>
-          <joint_control_type>position</joint_control_type>
-        </channel>
-        <channel name="tilt_unit4">
-          <input_index>16</input_index>
-          <input_offset>0</input_offset>
-          <input_scaling>${tilt_input_scaling}</input_scaling>
-          <zero_position_disarmed>0</zero_position_disarmed>
-          <zero_position_armed>0</zero_position_armed>
-          <joint_control_type>position</joint_control_type>
-        </channel>
-        <channel name="tilt_unit5">
-          <input_index>17</input_index>
           <input_offset>0</input_offset>
           <input_scaling>${tilt_input_scaling}</input_scaling>

Commit message: added rotor configuration and fixed d_gain error

File: rotors_description/urdf/griffin.xacro (robot description, xacro)
@@ -24,5 +24,5 @@
     <xacro:property name="use_mesh_file_core" value="true"/>
     <xacro:property name="use_mesh_file_rotor_unit" value="true"/>
-    <xacro:property name="mesh_file_core" value="package://rotors_description/meshes/test.dae"/>
+    <xacro:property name="mesh_file_core" value="package://rotors_description/meshes/sketch.dae"/>
     <xacro:property name="mesh_file_tilt_unit" value="package://rotors_description/meshes/omav/omav_tiltarm.dae"/>-->
     <xacro:property name="mass_core" value="2.30"/>    <!-- [kg] -->
@@ -31,6 +31,6 @@
     <xacro:property name="body_height" value="0.35"/>    <!-- [m] -->
     <xacro:property name="mass_rotor" value="0.0065"/>    <!-- [kg] -->
-    <xacro:property name="arm_length_front" value="0.600"/>    <!-- [m] -->
-    <xacro:property name="arm_length_back" value="0.4"/>
+    <xacro:property name="arm_length_front" value="0.4"/>    <!-- [m] -->
+    <xacro:property name="arm_length_back" value="0.6"/>
     <xacro:property name="rotor_offset_top" value="0.060"/>    <!-- [m] -->
     <xacro:property name="radius_rotor" value="0.1143"/>    <!-- [m] -->
@@ -106,5 +106,5 @@
     i_gain="${tilt_i_gain}"
     d_gain="${tilt_d_gain}">
-    <origin xyz="0 -${arm_length_front*sin60} ${arm_length_front*cos60}" rpy="-1.0471975512 0 0"/>
+    <origin xyz="${arm_length_front} 0 0" rpy="0 0 0"/>
     <xacro:insert_block name="rotor_inertia" />
   </xacro:double_tilt_unit>
@@ -134,5 +134,5 @@
     i_gain="${tilt_i_gain}"
     d_gain="${tilt_d_gain}">
-    <origin xyz="0 ${arm_length_front*sin60} ${arm_length_front*cos60}" rpy="1.0471975512 0 0"/>
+    <origin xyz="-${arm_length_front*cos60} ${arm_length_front*sin60} 0" rpy="0 0 2.09439510239"/>
     <xacro:insert_block name="rotor_inertia" />
   </xacro:double_tilt_unit>
@@ -162,5 +162,5 @@
     i_gain="${tilt_i_gain}"
     d_gain="${tilt_d_gain}">
-    <origin xyz="0 0 ${arm_length_front}" rpy="0 0 3.14159265359"/>
+    <origin xyz="-${arm_length_front*cos60} -${arm_length_front*sin60} 0" rpy="0 0 -2.09439510239"/>
     <xacro:insert_block name="rotor_inertia" />
   </xacro:double_tilt_unit>
@@ -189,5 +189,5 @@
     i_gain="${tilt_i_gain}"
     d_gain="${tilt_d_gain}">
-    <origin xyz="-${arm_length_back} 0 0" rpy="0 0 3.14159265359"/>
+    <origin xyz="0 0 ${arm_length_back}" rpy="0 -1.57079632679 0"/>
     <xacro:insert_block name="rotor_inertia" />
   </xacro:double_tilt_unit>

File: rotors_description/urdf/overactuated_base.xacro (robot description, xacro)
@@ -160,5 +160,5 @@
   <!-- Double tilt unit joint and link -->
   <xacro:macro name="double_tilt_unit"
-    params="robot_namespace suffix direction_upper direction_lower motor_constant motor_constant_lower moment_constant moment_constant_lower parent mass_rotor mass_tilt_unit time_constant_up time_constant_down max_rot_velocity rotor_offset_top motor_number rotor_drag_coefficient rolling_moment_coefficient color mesh mesh_tilt_unit *origin *inertia">
+    params="robot_namespace suffix direction_upper direction_lower motor_constant motor_constant_lower moment_constant moment_constant_lower parent mass_rotor mass_tilt_unit time_constant_up time_constant_down max_rot_velocity rotor_offset_top motor_number rotor_drag_coefficient rolling_moment_coefficient color mesh mesh_tilt_unit p_gain i_gain d_gain *origin *inertia">
     <!-- Rotor tilt_unit -->
     <joint name="${robot_namespace}/tilt_unit_${motor_number}_revolutejoint" type="continuous">
@@ -197,7 +197,7 @@
         <motorPositionPubTopic>/tilt_motor_${motor_number}/position</motorPositionPubTopic>
         <joint_control_pid>
-            <p>1.0</p>
-            <i>0.0</i>
-            <d>0.01</d>
+            <p>${p_gain}</p>
+            <i>${i_gain}</i>
+            <d>${d_gain}</d>
             <iMax>1.0</iMax>
             <iMin>-1.0</iMin>

Commit message: added gazebo plugins (doesn't seem to compile)

File: rotors_description/urdf/griffin.xacro (robot description, xacro)
@@ -234,37 +234,37 @@
         </channel>
         <channel name="rotor4">
+          <input_index>0</input_index>
+          <input_offset>0</input_offset>
+          <input_scaling>${max_rot_velocity}</input_scaling>
+          <zero_position_disarmed>0</zero_position_disarmed>
+          <zero_position_armed>100</zero_position_armed>
+          <joint_control_type>velocity</joint_control_type>
+        </channel>
+        <channel name="rotor5">
+          <input_index>1</input_index>
+          <input_offset>0</input_offset>
+          <input_scaling>${max_rot_velocity}</input_scaling>
+          <zero_position_disarmed>0</zero_position_disarmed>
+          <zero_position_armed>100</zero_position_armed>
+          <joint_control_type>velocity</joint_control_type>
+        </channel>
+         <channel name="rotor6">
+          <input_index>2</input_index>
+          <input_offset>0</input_offset>
+          <input_scaling>${max_rot_velocity}</input_scaling>
+          <zero_position_disarmed>0</zero_position_disarmed>
+          <zero_position_armed>100</zero_position_armed>
+          <joint_control_type>velocity</joint_control_type>
+        </channel>
+        <channel name="rotor7">
+          <input_index>3</input_index>
+          <input_offset>0</input_offset>
+          <input_scaling>${max_rot_velocity}</input_scaling>
+          <zero_position_disarmed>0</zero_position_disarmed>
+          <zero_position_armed>100</zero_position_armed>
+          <joint_control_type>velocity</joint_control_type>
+        </channel>
+        <channel name="tilt_unit0">
           <input_index>4</input_index>
-          <input_offset>0</input_offset>
-          <input_scaling>${max_rot_velocity}</input_scaling>
-          <zero_position_disarmed>0</zero_position_disarmed>
-          <zero_position_armed>100</zero_position_armed>
-          <joint_control_type>velocity</joint_control_type>
-        </channel>
-        <channel name="rotor5">
-          <input_index>5</input_index>
-          <input_offset>0</input_offset>
-          <input_scaling>${max_rot_velocity}</input_scaling>
-          <zero_position_disarmed>0</zero_position_disarmed>
-          <zero_position_armed>100</zero_position_armed>
-          <joint_control_type>velocity</joint_control_type>
-        </channel>
-         <channel name="rotor6">
-          <input_index>6</input_index>
-          <input_offset>0</input_offset>
-          <input_scaling>${max_rot_velocity}</input_scaling>
-          <zero_position_disarmed>0</zero_position_disarmed>
-          <zero_position_armed>100</zero_position_armed>
-          <joint_control_type>velocity</joint_control_type>
-        </channel>
-        <channel name="rotor7">
-          <input_index>7</input_index>
-          <input_offset>0</input_offset>
-          <input_scaling>${max_rot_velocity}</input_scaling>
-          <zero_position_disarmed>0</zero_position_disarmed>
-          <zero_position_armed>100</zero_position_armed>
-          <joint_control_type>velocity</joint_control_type>
-        </channel>
-        <channel name="tilt_unit0">
-          <input_index>12</input_index>
           <input_offset>0</input_offset>
           <input_scaling>${tilt_input_scaling}</input_scaling>
@@ -274,5 +274,5 @@
         </channel>
         <channel name="tilt_unit1">
-          <input_index>13</input_index>
+          <input_index>5</input_index>
           <input_offset>0</input_offset>
           <input_scaling>${tilt_input_scaling}</input_scaling>
@@ -282,5 +282,5 @@
         </channel>
         <channel name="tilt_unit2">
-          <input_index>14</input_index>
+          <input_index>6</input_index>
           <input_offset>0</input_offset>
           <input_scaling>${tilt_input_scaling}</input_scaling>
@@ -290,5 +290,5 @@
         </channel>
         <channel name="tilt_unit3">
-          <input_index>15</input_index>
+          <input_index>7</input_index>
           <input_offset>0</input_offset>
           <input_scaling>${tilt_input_scaling}</input_scaling>

File: rotors_description/urdf/overactuated_base.xacro (robot description, xacro)
@@ -257,11 +257,11 @@
     </gazebo>
     <!-- Lower Rotor -->
-    <joint name="rotor_${motor_number+6}_joint" type="continuous">
+    <joint name="rotor_${motor_number+4}_joint" type="continuous">
       <origin xyz="0 0 ${-rotor_offset_top}" rpy="0 0 0" />
       <axis xyz="0 0 1" />
       <parent link="${namespace}/tilt_unit_${motor_number}" />
-      <child link="rotor_${motor_number+6}" />
-    </joint>
-    <link name="rotor_${motor_number+6}">
+      <child link="rotor_${motor_number+4}" />
+    </joint>
+    <link name="rotor_${motor_number+4}">
       <inertial>
         <mass value="${mass_rotor}" /> <!-- [kg] -->
@@ -283,6 +283,6 @@
       <plugin name="${suffix}_lower_motor_model" filename="librotors_gazebo_motor_model.so">
         <robotNamespace>${robot_namespace}</robotNamespace>
-        <jointName>rotor_${motor_number+6}_joint</jointName>
-        <linkName>rotor_${motor_number+6}</linkName>
+        <jointName>rotor_${motor_number+4}_joint</jointName>
+        <linkName>rotor_${motor_number+4}</linkName>
         <turningDirection>${direction_lower}</turningDirection>
         <timeConstantUp>${time_constant_up}</timeConstantUp>
@@ -292,5 +292,5 @@
         <momentConstant>${moment_constant_lower}</momentConstant>
         <commandSubTopic>/gazebo/command/motor_speed</commandSubTopic>
-        <motorNumber>${motor_number+6}</motorNumber>
+        <motorNumber>${motor_number+4}</motorNumber>
         <rotorDragCoefficient>${rotor_drag_coefficient}</rotorDragCoefficient>
         <rollingMomentCoefficient>${rolling_moment_coefficient}</rollingMomentCoefficient>
@@ -299,5 +299,5 @@
       </plugin>
     </gazebo>
-    <gazebo reference="rotor_${motor_number+6}">
+    <gazebo reference="rotor_${motor_number+4}">
       <material>Gazebo/${color}</material>
     </gazebo>
