Commit message: updated xacro-file according to omav3

File: rotors_description/urdf/griffin_base.xacro (robot description, xacro)
@@ -1,39 +1,61 @@
 <?xml version="1.0"?>
-<!--
-  Copyright 2015 Fadri Furrer, ASL, ETH Zurich, Switzerland
-  Copyright 2015 Michael Burri, ASL, ETH Zurich, Switzerland
-  Copyright 2015 Mina Kamel, ASL, ETH Zurich, Switzerland
-  Copyright 2015 Janosch Nikolic, ASL, ETH Zurich, Switzerland
-  Copyright 2015 Markus Achtelik, ASL, ETH Zurich, Switzerland
-  Licensed under the Apache License, Version 2.0 (the "License");
-  you may not use this file except in compliance with the License.
-  You may obtain a copy of the License at
-  http://www.apache.org/licenses/LICENSE-2.0
-  Unless required by applicable law or agreed to in writing, software
-  distributed under the License is distributed on an "AS IS" BASIS,
-  WITHOUT WARRANTIES OR CONDITIONS OF ANY KIND, either express or implied.
-  See the License for the specific language governing permissions and
-  limitations under the License.
--->
-<robot name="griffin" xmlns:xacro="http://ros.org/wiki/xacro">
-  <xacro:include filename="$(find rotors_description)/urdf/component_snippets.xacro"/>
-  <!-- Instantiate OMAV "mechanics". -->
-  <xacro:include filename="$(find rotors_description)/urdf/griffin.xacro"/>
-  <!-- Instantiate a controller. -->
-  <xacro:controller_plugin_macro namespace="${namespace}" imu_sub_topic="imu"/>
-  <!-- Mount an ADIS16448 IMU. -->
-  <xacro:default_imu namespace="${namespace}" parent_link="${namespace}/base_link"/>
-  <xacro:if value="$(arg enable_ground_truth)">
-      <xacro:ground_truth_imu_and_odometry
-        namespace="${namespace}"
-        parent_link="${namespace}/base_link"/>
-  </xacro:if>
-  <xacro:if value="$(arg enable_logging)">
-      <!-- Instantiate a logger. -->
-      <xacro:bag_plugin_macro
-        namespace="${namespace}"
-        bag_file="$(arg log_file)"
-        rotor_velocity_slowdown_sim="${rotor_velocity_slowdown_sim}"
-        wait_to_record_bag="$(arg wait_to_record_bag)"/>
-  </xacro:if>
+<robot name="$(arg mav_name)" xmlns:xacro="http://ros.org/wiki/xacro">
+    <xacro:include filename="$(find rotors_description)/urdf/component_snippets.xacro"/>
+    <xacro:property name="mounting_roll" value="$(arg model_roll)" />
+    <!-- Instantiate OMAV "mechanics". -->
+    <xacro:include filename="$(find rotors_description)/urdf/griffin.xacro"/>
+    <!-- Add manipulator. -->
+    <xacro:if value="$(arg add_manipulator)">
+        <xacro:property name="robot_name" value="delta" />
+        <xacro:property name="delta_namespace" value="delta" />
+        <xacro:property name="mounting_link" value="$(arg mav_name)/base_link" />
+        <xacro:property name="height_offset" value="0.073" />
+        <xacro:include filename="$(find rotors_description)/urdf/delta_manipulator.xacro" />
+        <xacro:include filename="$(find rotors_description)/urdf/delta_actuators.xacro" />
+    </xacro:if>
+    <xacro:include filename="$(find rotors_description)/urdf/griffin_actuators.xacro" />
+    <!-- Mount an ADIS16448 IMU. -->
+    <!-- Note that the gyroscope_noise_density is not the discrete noise density used in the simulation. In gazebo_imu_plugin, the discrete noise density is computed as 1/sqrt(dt)*gyroscope_noise_density, where dt the time step in simulation -->
+    <xacro:imu_plugin_macro
+            namespace="$(arg mav_name)"
+            imu_suffix=""
+            parent_link="$(arg mav_name)/base_link_inertia"
+            imu_topic="imu"
+            mass_imu_sensor="0.015"
+            gyroscope_noise_density="0.00005366563"
+            gyroscope_random_walk="0.000038785"
+            gyroscope_bias_correlation_time="1000.0"
+            gyroscope_turn_on_bias_sigma="0.0087"
+            accelerometer_noise_density="0.004"
+            accelerometer_random_walk="0.006"
+            accelerometer_bias_correlation_time="300.0"
+            accelerometer_turn_on_bias_sigma="0.1960"
+            measurement_divisor="2">
+        <inertia ixx="0.00001" ixy="0.0" ixz="0.0" iyy="0.00001" iyz="0.0" izz="0.00001" />
+        <origin xyz="0 0 0" rpy="0 0 0" />
+    </xacro:imu_plugin_macro>
+    <xacro:if value="$(arg enable_ground_truth)">
+        <xacro:ground_truth_imu_and_odometry
+                namespace="$(arg mav_name)"
+                parent_link="$(arg mav_name)/base_link_inertia"/>
+    </xacro:if>
+    <xacro:if value="$(arg enable_logging)">
+        <!-- Instantiate a logger. -->
+        <xacro:bag_plugin_macro
+                namespace="$(arg mav_name)"
+                bag_file="$(arg log_file)"
+                rotor_velocity_slowdown_sim="${rotor_velocity_slowdown_sim}"
+                wait_to_record_bag="$(arg wait_to_record_bag)"/>
+    </xacro:if>
+    <xacro:if value="$(arg add_rgbd_sensor)">
+        <!-- Add a RGB-D sensor -->
+        <xacro:include filename="$(find rotors_description)/urdf/pmd_monstar.xacro"/>
+        <joint name="$(arg mav_name)/tof_cam_optical_frame" type="fixed">
+            <origin xyz="0.09 0.0 0.15" rpy="-1.309 0 -1.571"/>
+            <parent link="$(arg mav_name)/base_link_inertia" />
+            <child link="rgbd_camera/base_link" />
+        </joint>
+    </xacro:if>
+    <!-- Add odometry. -->
+    <xacro:include filename="$(find rotors_description)/urdf/odometry_sensor_smooth.xacro"/>
 </robot>

Commit message: added double_tilt_unit_minimal and updated urdf

File: rotors_description/urdf/griffin.xacro (robot description, xacro)
@@ -69,7 +69,10 @@
           body_width="${body_width}"
           body_height="${body_height}"
-          use_mesh_file="${use_mesh_file_core}"
+          use_mesh_file="false"
+          mesh_file="false"
+          collision_mesh_file="false">
+         <!-- use_mesh_file="${use_mesh_file_core}"
           mesh_file="${mesh_file_core}"
-          collision_mesh_file="${mesh_file_core_collision}">
+          collision_mesh_file="${mesh_file_core_collision}"-->
     <xacro:insert_block name="body_origin"/>
     <xacro:insert_block name="body_inertia"/>
@@ -78,7 +81,8 @@
   <!-- Instantiate rotors -->
   <!-- front0-->
-  <xacro:single_tilt_unit_minimal
+  <xacro:double_tilt_unit_minimal
           robot_namespace="${namespace}"
-          direction="ccw"
+          direction_upper="ccw"
+          direction_lower="cw"
           parent="${tilt_unit_parent}"
           mass_rotor="${mass_rotor}"
@@ -91,9 +95,10 @@
     <origin xyz="${arm_length_front} 0 0" rpy="0 0 0"/>
     <xacro:insert_block name="rotor_inertia" />
-  </xacro:single_tilt_unit_minimal>
+  </xacro:double_tilt_unit_minimal>
   <!-- front1 -->
-  <xacro:single_tilt_unit_minimal
+  <xacro:double_tilt_unit_minimal
           robot_namespace="${namespace}"
-          direction="cw"
+          direction_upper="ccw"
+          direction_lower="cw"
           parent="${tilt_unit_parent}"
           mass_rotor="${mass_rotor}"
@@ -106,9 +111,10 @@
     <origin xyz="-${arm_length_front*cos60} ${arm_length_front*sin60} 0" rpy="0 0 2.09439510239"/>
     <xacro:insert_block name="rotor_inertia" />
-  </xacro:single_tilt_unit_minimal>
+  </xacro:double_tilt_unit_minimal>
   <!-- front2 -->
-  <xacro:single_tilt_unit_minimal
+  <xacro:double_tilt_unit_minimal
           robot_namespace="${namespace}"
-          direction="ccw"
+          direction_upper="ccw"
+          direction_lower="cw"
           parent="${tilt_unit_parent}"
           mass_rotor="${mass_rotor}"
@@ -121,9 +127,10 @@
     <origin xyz="-${arm_length_front*cos60} -${arm_length_front*sin60} 0" rpy="0 0 -2.09439510239"/>
     <xacro:insert_block name="rotor_inertia" />
-  </xacro:single_tilt_unit_minimal>
+  </xacro:double_tilt_unit_minimal>
   <!-- back3 -->
-  <xacro:single_tilt_unit_minimal
+  <xacro:double_tilt_unit_minimal
           robot_namespace="${namespace}"
-          direction="cw"
+          direction_upper="ccw"
+          direction_lower="cw"
           parent="${tilt_unit_parent}"
           mass_rotor="${mass_rotor}"
@@ -136,4 +143,4 @@
     <origin xyz="0 0 ${arm_length_back}" rpy="0 -1.57079632679 0"/>
     <xacro:insert_block name="rotor_inertia" />
-  </xacro:single_tilt_unit_minimal>
+  </xacro:double_tilt_unit_minimal>
 </robot>

File: rotors_description/urdf/griffin_actuators.xacro (robot description, xacro)
@@ -26,20 +26,20 @@
         <rotors>
             <rotor>
-              <jointName>rotor_0_joint</jointName>
-              <linkName>rotor_0</linkName>
-              <spinDirection>ccw</spinDirection>
-              <timeConstantUp>${time_constant_up}</timeConstantUp>
-              <timeConstantDown>${time_constant_down}</timeConstantDown>
-              <minRotVelocity>${min_rot_velocity}</minRotVelocity>
-              <maxRotVelocity>${max_rot_velocity}</maxRotVelocity>
-              <thrustConstant>${motor_constant}</thrustConstant>
-              <momentConstant>${moment_constant}</momentConstant>
-              <rotorDragCoefficient>${rotor_drag_coefficient}</rotorDragCoefficient>
-              <rollingMomentCoefficient>${rolling_moment_coefficient}</rollingMomentCoefficient>
-              <rotorVelocitySlowdownSim>${rotor_velocity_slowdown_sim}</rotorVelocitySlowdownSim>
-            </rotor>
-            <rotor>
-              <jointName>rotor_1_joint</jointName>
-              <linkName>rotor_1</linkName>
+              <jointName>rotor_01_joint</jointName>
+              <linkName>rotor_01</linkName>
+              <spinDirection>ccw</spinDirection>
+              <timeConstantUp>${time_constant_up}</timeConstantUp>
+              <timeConstantDown>${time_constant_down}</timeConstantDown>
+              <minRotVelocity>${min_rot_velocity}</minRotVelocity>
+              <maxRotVelocity>${max_rot_velocity}</maxRotVelocity>
+              <thrustConstant>${motor_constant}</thrustConstant>
+              <momentConstant>${moment_constant}</momentConstant>
+              <rotorDragCoefficient>${rotor_drag_coefficient}</rotorDragCoefficient>
+              <rollingMomentCoefficient>${rolling_moment_coefficient}</rollingMomentCoefficient>
+              <rotorVelocitySlowdownSim>${rotor_velocity_slowdown_sim}</rotorVelocitySlowdownSim>
+            </rotor>
+            <rotor>
+              <jointName>rotor_02_joint</jointName>
+              <linkName>rotor_02</linkName>
               <spinDirection>cw</spinDirection>
               <timeConstantUp>${time_constant_up}</timeConstantUp>
@@ -54,20 +54,20 @@
             </rotor>
             <rotor>
-              <jointName>rotor_2_joint</jointName>
-              <linkName>rotor_2</linkName>
-              <spinDirection>ccw</spinDirection>
-              <timeConstantUp>${time_constant_up}</timeConstantUp>
-              <timeConstantDown>${time_constant_down}</timeConstantDown>
-              <minRotVelocity>${min_rot_velocity}</minRotVelocity>
-              <maxRotVelocity>${max_rot_velocity}</maxRotVelocity>
-              <thrustConstant>${motor_constant}</thrustConstant>
-              <momentConstant>${moment_constant}</momentConstant>
-              <rotorDragCoefficient>${rotor_drag_coefficient}</rotorDragCoefficient>
-              <rollingMomentCoefficient>${rolling_moment_coefficient}</rollingMomentCoefficient>
-              <rotorVelocitySlowdownSim>${rotor_velocity_slowdown_sim}</rotorVelocitySlowdownSim>
-            </rotor>
-            <rotor>
-              <jointName>rotor_3_joint</jointName>
-              <linkName>rotor_3</linkName>
+              <jointName>rotor_11_joint</jointName>
+              <linkName>rotor_11</linkName>
+              <spinDirection>ccw</spinDirection>
+              <timeConstantUp>${time_constant_up}</timeConstantUp>
+              <timeConstantDown>${time_constant_down}</timeConstantDown>
+              <minRotVelocity>${min_rot_velocity}</minRotVelocity>
+              <maxRotVelocity>${max_rot_velocity}</maxRotVelocity>
+              <thrustConstant>${motor_constant}</thrustConstant>
+              <momentConstant>${moment_constant}</momentConstant>
+              <rotorDragCoefficient>${rotor_drag_coefficient}</rotorDragCoefficient>
+              <rollingMomentCoefficient>${rolling_moment_coefficient}</rollingMomentCoefficient>
+              <rotorVelocitySlowdownSim>${rotor_velocity_slowdown_sim}</rotorVelocitySlowdownSim>
+            </rotor>
+            <rotor>
+              <jointName>rotor_12_joint</jointName>
+              <linkName>rotor_12</linkName>
               <spinDirection>cw</spinDirection>
               <timeConstantUp>${time_constant_up}</timeConstantUp>
@@ -80,4 +80,60 @@
               <rollingMomentCoefficient>${rolling_moment_coefficient}</rollingMomentCoefficient>
               <rotorVelocitySlowdownSim>${rotor_velocity_slowdown_sim}</rotorVelocitySlowdownSim>
+            </rotor>
+            <rotor>
+                <jointName>rotor_21_joint</jointName>
+                <linkName>rotor_21</linkName>
+                <spinDirection>ccw</spinDirection>
+                <timeConstantUp>${time_constant_up}</timeConstantUp>
+                <timeConstantDown>${time_constant_down}</timeConstantDown>
+                <minRotVelocity>${min_rot_velocity}</minRotVelocity>
+                <maxRotVelocity>${max_rot_velocity}</maxRotVelocity>
+                <thrustConstant>${motor_constant}</thrustConstant>
+                <momentConstant>${moment_constant}</momentConstant>
+                <rotorDragCoefficient>${rotor_drag_coefficient}</rotorDragCoefficient>
+                <rollingMomentCoefficient>${rolling_moment_coefficient}</rollingMomentCoefficient>
+                <rotorVelocitySlowdownSim>${rotor_velocity_slowdown_sim}</rotorVelocitySlowdownSim>
+            </rotor>
+            <rotor>
+                <jointName>rotor_22_joint</jointName>
+                <linkName>rotor_22</linkName>
+                <spinDirection>cw</spinDirection>
+                <timeConstantUp>${time_constant_up}</timeConstantUp>
+                <timeConstantDown>${time_constant_down}</timeConstantDown>
+                <minRotVelocity>${min_rot_velocity}</minRotVelocity>
+                <maxRotVelocity>${max_rot_velocity}</maxRotVelocity>
+                <thrustConstant>${motor_constant}</thrustConstant>
+                <momentConstant>${moment_constant}</momentConstant>
+                <rotorDragCoefficient>${rotor_drag_coefficient}</rotorDragCoefficient>
+                <rollingMomentCoefficient>${rolling_moment_coefficient}</rollingMomentCoefficient>
+                <rotorVelocitySlowdownSim>${rotor_velocity_slowdown_sim}</rotorVelocitySlowdownSim>
+            </rotor>
+            <rotor>
+                <jointName>rotor_31_joint</jointName>
+                <linkName>rotor_31</linkName>
+                <spinDirection>ccw</spinDirection>
+                <timeConstantUp>${time_constant_up}</timeConstantUp>
+                <timeConstantDown>${time_constant_down}</timeConstantDown>
+                <minRotVelocity>${min_rot_velocity}</minRotVelocity>
+                <maxRotVelocity>${max_rot_velocity}</maxRotVelocity>
+                <thrustConstant>${motor_constant}</thrustConstant>
+                <momentConstant>${moment_constant}</momentConstant>
+                <rotorDragCoefficient>${rotor_drag_coefficient}</rotorDragCoefficient>
+                <rollingMomentCoefficient>${rolling_moment_coefficient}</rollingMomentCoefficient>
+                <rotorVelocitySlowdownSim>${rotor_velocity_slowdown_sim}</rotorVelocitySlowdownSim>
+            </rotor>
+            <rotor>
+                <jointName>rotor_32_joint</jointName>
+                <linkName>rotor_32</linkName>
+                <spinDirection>cw</spinDirection>
+                <timeConstantUp>${time_constant_up}</timeConstantUp>
+                <timeConstantDown>${time_constant_down}</timeConstantDown>
+                <minRotVelocity>${min_rot_velocity}</minRotVelocity>
+                <maxRotVelocity>${max_rot_velocity}</maxRotVelocity>
+                <thrustConstant>${motor_constant}</thrustConstant>
+                <momentConstant>${moment_constant}</momentConstant>
+                <rotorDragCoefficient>${rotor_drag_coefficient}</rotorDragCoefficient>
+                <rollingMomentCoefficient>${rolling_moment_coefficient}</rollingMomentCoefficient>
+                <rotorVelocitySlowdownSim>${rotor_velocity_slowdown_sim}</rotorVelocitySlowdownSim>
             </rotor>
         </rotors>

File: rotors_description/urdf/omav_snippets.xacro (robot description, xacro)
@@ -246,7 +246,7 @@
     </gazebo>
   </xacro:macro>
-  <!-- Double tilt unit joint and link -->
-  <xacro:macro name="double_tilt_unit"
-    params="robot_namespace suffix direction_upper direction_lower motor_constant motor_constant_lower moment_constant moment_constant_lower parent mass_rotor mass_tilt_unit time_constant_up time_constant_down max_rot_velocity rotor_offset_top motor_number rotor_drag_coefficient rolling_moment_coefficient color mesh mesh_tilt_unit p_gain i_gain d_gain *origin *inertia">
+  <!-- Double tilt unit minimal-->
+  <xacro:macro name="double_tilt_unit_minimal"
+               params="robot_namespace direction_upper direction_lower parent mass_rotor mass_tilt_unit rotor_offset_top motor_number color mesh mesh_tilt_unit *origin *inertia">
     <!-- Rotor tilt_unit -->
     <joint name="${robot_namespace}/tilt_unit_${motor_number}_revolutejoint" type="continuous">
@@ -256,4 +256,7 @@
       <child link="${namespace}/tilt_unit_${motor_number}" />
     </joint>
+    <gazebo reference="${robot_namespace}/tilt_unit_${motor_number}_revolutejoint">
+      <provideFeedback>true</provideFeedback>
+    </gazebo>
     <link name="${namespace}/tilt_unit_${motor_number}">
       <inertial>
@@ -263,6 +266,91 @@
       <visual>
         <geometry>
-            <mesh filename="${mesh_tilt_unit}"
-              scale="1 1 1" />
+          <mesh filename="${mesh_tilt_unit}"
+                scale="1 1 1" />
+        </geometry>
+      </visual>
+      <collision>
+        <geometry>
+          <box size="0.005 0.005 0.005"  /> <!-- [m] -->
+        </geometry>
+      </collision>
+    </link>
+    <gazebo reference="${namespace}/tilt_unit_${motor_number}">
+      <material>Gazebo/White</material>
+    </gazebo>
+    <!-- Upper Rotor -->
+    <joint name="rotor_${motor_number}1_joint" type="continuous">
+      <origin xyz="0 0 ${rotor_offset_top}" rpy="0 0 0" />
+      <axis xyz="0 0 1" />
+      <parent link="${namespace}/tilt_unit_${motor_number}" />
+      <child link="rotor_${motor_number}1" />
+    </joint>
+    <link name="rotor_${motor_number}1">
+      <inertial>
+        <mass value="${mass_rotor}" /> <!-- [kg] -->
+        <xacro:insert_block name="inertia" />
+      </inertial>
+      <visual>
+        <geometry>
+          <mesh filename="package://rotors_description/meshes/${mesh}_${direction_upper}.dae"
+                scale="${radius_rotor} ${radius_rotor} ${radius_rotor}" />
+        </geometry>
+      </visual>
+      <collision>
+        <geometry>
+          <cylinder length="0.005" radius="${radius_rotor}" /> <!-- [m] -->
+        </geometry>
+      </collision>
+    </link>
+    <gazebo reference="rotor_${motor_number}1">
+      <material>Gazebo/${color}</material>
+    </gazebo>
+    <!-- Lower Rotor -->
+    <joint name="rotor_${motor_number}2_joint" type="continuous">
+      <origin xyz="0 0 ${-rotor_offset_top}" rpy="0 0 0" />
+      <axis xyz="0 0 1" />
+      <parent link="${namespace}/tilt_unit_${motor_number}" />
+      <child link="rotor_${motor_number}2" />
+    </joint>
+    <link name="rotor_${motor_number}2">
+      <inertial>
+        <mass value="${mass_rotor}" /> <!-- [kg] -->
+        <xacro:insert_block name="inertia" />
+      </inertial>
+      <visual>
+        <geometry>
+          <mesh filename="package://rotors_description/meshes/${mesh}_${direction_lower}.dae"
+                scale="${radius_rotor} ${radius_rotor} ${radius_rotor}" />
+        </geometry>
+      </visual>
+      <collision>
+        <geometry>
+          <cylinder length="0.005" radius="${radius_rotor}" /> <!-- [m] -->
+        </geometry>
+      </collision>
+    </link>
+    <gazebo reference="rotor_${motor_number}2">
+      <material>Gazebo/${color}</material>
+    </gazebo>
+  </xacro:macro>
+  <!-- Double tilt unit joint and link -->
+  <xacro:macro name="double_tilt_unit"
+               params="robot_namespace suffix direction_upper direction_lower motor_constant motor_constant_lower moment_constant moment_constant_lower parent mass_rotor mass_tilt_unit time_constant_up time_constant_down max_rot_velocity rotor_offset_top motor_number rotor_drag_coefficient rolling_moment_coefficient color mesh mesh_tilt_unit p_gain i_gain d_gain *origin *inertia">
+    <!-- Rotor tilt_unit -->
+    <joint name="${robot_namespace}/tilt_unit_${motor_number}_revolutejoint" type="continuous">
+      <xacro:insert_block name="origin" />
+      <axis xyz="1 0 0" />
+      <parent link="${parent}" />
+      <child link="${namespace}/tilt_unit_${motor_number}" />
+    </joint>
+    <link name="${namespace}/tilt_unit_${motor_number}">
+      <inertial>
+        <mass value="${mass_tilt_unit}" /> <!-- [kg] -->
+        <xacro:insert_block name="tilt_unit_inertia" />
+      </inertial>
+      <visual>
+        <geometry>
+          <mesh filename="${mesh_tilt_unit}"
+                scale="1 1 1" />
         </geometry>
       </visual>
@@ -285,11 +373,11 @@
         <motorPositionPubTopic>/tilt_motor_${motor_number}/position</motorPositionPubTopic>
         <joint_control_pid>
-            <p>${p_gain}</p>
-            <i>${i_gain}</i>
-            <d>${d_gain}</d>
-            <iMax>1.0</iMax>
-            <iMin>-1.0</iMin>
-            <cmdMax>2.0</cmdMax>
-            <cmdMin>-2.0</cmdMin>
+          <p>${p_gain}</p>
+          <i>${i_gain}</i>
+          <d>${d_gain}</d>
+          <iMax>1.0</iMax>
+          <iMin>-1.0</iMin>
+          <cmdMax>2.0</cmdMax>
+          <cmdMin>-2.0</cmdMin>
         </joint_control_pid>
       </plugin>
@@ -313,5 +401,5 @@
         <geometry>
           <mesh filename="package://rotors_description/meshes/${mesh}_${direction_upper}.dae"
-            scale="${radius_rotor} ${radius_rotor} ${radius_rotor}" />
+                scale="${radius_rotor} ${radius_rotor} ${radius_rotor}" />
         </geometry>
       </visual>
@@ -359,5 +447,5 @@
         <geometry>
           <mesh filename="package://rotors_description/meshes/${mesh}_${direction_lower}.dae"
-            scale="${radius_rotor} ${radius_rotor} ${radius_rotor}" />
+                scale="${radius_rotor} ${radius_rotor} ${radius_rotor}" />
         </geometry>
       </visual>
