Commit message: added stl-file of body and tilt-unit

File: rotors_description/urdf/griffin.xacro (robot description, xacro)
@@ -24,15 +24,15 @@
   <xacro:property name="use_mesh_file_core" value="true"/>
   <xacro:property name="use_mesh_file_rotor_unit" value="true"/>
-  <xacro:property name="mesh_file_core" value="package://rotors_description/meshes/omav/omav3_base.stl"/>
-  <xacro:property name="mesh_file_core_collision" value="package://rotors_description/meshes/omav/omav3_base.stl"/>
-  <xacro:property name="mesh_file_tilt_unit" value="package://rotors_description/meshes/omav/omav3_tiltarm.stl"/>
+  <xacro:property name="mesh_file_core" value="package://rotors_description/meshes/omav/griffin_base.stl"/>
+  <xacro:property name="mesh_file_core_collision" value="package://rotors_description/meshes/omav/griffin_base.stl"/>
+  <xacro:property name="mesh_file_tilt_unit" value="package://rotors_description/meshes/omav/griffin_tilt_unit.stl"/>
   <xacro:property name="mass_core" value="3.13"/>    <!-- [kg] -->
   <xacro:property name="mass_tilt_unit" value="0.277"/>    <!-- [kg] -->
   <xacro:property name="body_width" value="0.22"/>    <!-- [m] -->
-  <xacro:property name="body_height" value="0.45"/>    <!-- [m] -->
+  <xacro:property name="body_height" value="0.666"/>    <!-- [m] -->
   <xacro:property name="mass_rotor" value="0.0065"/>    <!-- [kg] -->
-  <xacro:property name="arm_length_front" value="0.3"/> <!-- [m] -->
-  <xacro:property name="arm_length_back" value="0.4"/> <!-- [m] -->
-  <xacro:property name="rotor_offset_top" value="0.035"/>    <!-- [m] -->
+  <xacro:property name="arm_length_front" value="0.37"/> <!-- [m] -->
+  <xacro:property name="arm_length_back" value="0.6"/> <!-- [m] -->
+  <xacro:property name="rotor_offset_top" value="0.045"/>    <!-- [m] -->
   <xacro:property name="radius_rotor" value="${0.1143*4/3}"/>    <!-- 12 in [m] -->
   <xacro:property name="tilt_unit_parent" value="${namespace}/base_link_inertia"/>    <!-- 12 in [m] -->
@@ -69,10 +69,7 @@
           body_width="${body_width}"
           body_height="${body_height}"
-          use_mesh_file="false"
-          mesh_file="false"
-          collision_mesh_file="false">
-         <!-- use_mesh_file="${use_mesh_file_core}"
+          use_mesh_file="${use_mesh_file_core}"
           mesh_file="${mesh_file_core}"
-          collision_mesh_file="${mesh_file_core_collision}"-->
+          collision_mesh_file="${mesh_file_core_collision}">
     <xacro:insert_block name="body_origin"/>
     <xacro:insert_block name="body_inertia"/>
@@ -93,5 +90,5 @@
           mesh_tilt_unit="${mesh_file_tilt_unit}"
           color="Black">
-    <origin xyz="${arm_length_front} 0 0" rpy="0 0 0"/>
+    <origin xyz="0 ${arm_length_front} 0" rpy="0 0 1.57079632679"/>
     <xacro:insert_block name="rotor_inertia" />
   </xacro:double_tilt_unit_minimal>
@@ -109,5 +106,5 @@
           mesh_tilt_unit="${mesh_file_tilt_unit}"
           color="Black">
-    <origin xyz="-${arm_length_front*cos60} ${arm_length_front*sin60} 0" rpy="0 0 2.09439510239"/>
+    <origin xyz="${arm_length_front*cos30} -${arm_length_front*sin30} 0" rpy="0 0 -0.52359877559"/>
     <xacro:insert_block name="rotor_inertia" />
   </xacro:double_tilt_unit_minimal>
@@ -125,5 +122,5 @@
           mesh_tilt_unit="${mesh_file_tilt_unit}"
           color="Orange">
-    <origin xyz="-${arm_length_front*cos60} -${arm_length_front*sin60} 0" rpy="0 0 -2.09439510239"/>
+    <origin xyz="-${arm_length_front*cos30} -${arm_length_front*sin30} 0" rpy="0 0 -2.61799387799"/>
     <xacro:insert_block name="rotor_inertia" />
   </xacro:double_tilt_unit_minimal>

Commit message: added geometrical values (inertia, mass...)

File: rotors_description/urdf/griffin.xacro (robot description, xacro)
@@ -27,13 +27,14 @@
   <xacro:property name="mesh_file_core_collision" value="package://rotors_description/meshes/omav/griffin_base.stl"/>
   <xacro:property name="mesh_file_tilt_unit" value="package://rotors_description/meshes/omav/griffin_tilt_unit.stl"/>
-  <xacro:property name="mass_core" value="3.13"/>    <!-- [kg] -->
-  <xacro:property name="mass_tilt_unit" value="0.277"/>    <!-- [kg] -->
-  <xacro:property name="body_width" value="0.22"/>    <!-- [m] -->
-  <xacro:property name="body_height" value="0.666"/>    <!-- [m] -->
-  <xacro:property name="mass_rotor" value="0.0065"/>    <!-- [kg] -->
-  <xacro:property name="arm_length_front" value="0.37"/> <!-- [m] -->
-  <xacro:property name="arm_length_back" value="0.6"/> <!-- [m] -->
-  <xacro:property name="rotor_offset_top" value="0.045"/>    <!-- [m] -->
-  <xacro:property name="radius_rotor" value="${0.1143*4/3}"/>    <!-- 12 in [m] -->
+  <xacro:property name="mass_core" value="6.57"/>    <!-- [kg] -->
+  <xacro:property name="mass_tilt_unit" value="0.33"/>    <!-- [kg] -->
+  <xacro:property name="body_width" value="0.22"/>    <!-- [m] TODO -->
+  <xacro:property name="body_height" value="0.666"/>    <!-- [m] TODO -->
+  <xacro:property name="mass_rotor" value="0.045"/>    <!-- [kg] -->
+  <xacro:property name="arm_length_front" value="0.35"/> <!-- [m] -->
+  <xacro:property name="arm_length_back" value="0.595"/> <!-- [m] -->
+  <xacro:property name="rotor_offset_top" value="0.0445"/>    <!-- [m] -->
+  <xacro:property name="radius_rotor" value="${0.406/2}"/>    <!-- 12 in [m] -->
+  <xacro:property name="mass_tilt_unit_back" value="0.32"/> <!-- [kg] -->
   <xacro:property name="tilt_unit_parent" value="${namespace}/base_link_inertia"/>    <!-- 12 in [m] -->
   <xacro:property name="body_origin">
@@ -46,5 +47,5 @@
   <!-- Property Blocks -->
   <xacro:property name="body_inertia">
-    <inertia ixx="0.0075" ixy="${-3.4208e-05}" ixz="${2.4695e-05}" iyy="0.010939" iyz="${-3.8826e-06}" izz="0.01369"/>
+    <inertia ixx="0.30015" ixy="${-6.707e-5}" ixz="${2.937e-3}" iyy="0.2979" iyz="${1.257e-5}" izz="0.04738"/>
     <!-- [kg m^2] [kg m^2] [kg m^2] [kg m^2] [kg m^2] [kg m^2] -->
   </xacro:property>
@@ -52,12 +53,12 @@
   <xacro:property name="body_inertia_origin">
     <!-- <origin xyz="0.03 0 0.01" /> -->
-    <origin xyz="0.0 0.0 0.0" />
+    <origin xyz="-0.0024 -0.0035 0.121" /> <!-- [m] -->
   </xacro:property>
   <!-- Rotor unit inertia without the propellor. -->
   <xacro:property name="tilt_unit_inertia">
-    <inertia ixx="0.00034257" ixy="0" ixz="0" iyy="0.0013205" iyz="0" izz="0.0010037"/>
+    <inertia ixx="${3.157e-4}" ixy="0" ixz="0" iyy="${1.795e-3}" iyz="0" izz="${2.025e-3}"/>
     <!-- [kg m^2] [kg m^2] [kg m^2] [kg m^2] [kg m^2] [kg m^2] -->
   </xacro:property>
-  <!-- Inertia of a single rotor, assuming it is a cuboid. Height=3mm, width=15mm. -->
+  <!-- Inertia of a single rotor, assuming it is a cuboid. Height=3mm, width=15mm. TODO -->
   <xacro:property name="rotor_inertia">
     <xacro:box_inertia x="${radius_rotor}" y="0.020" z="0.003" mass="${mass_rotor*rotor_velocity_slowdown_sim}"/>
@@ -132,5 +133,5 @@
           parent="${tilt_unit_parent}"
           mass_rotor="${mass_rotor}"
-          mass_tilt_unit="${mass_tilt_unit}"
+          mass_tilt_unit="${mass_tilt_unit_back}"
           rotor_offset_top="${rotor_offset_top}"
           motor_number="3"

File: rotors_description/urdf/griffin_actuators.xacro (robot description, xacro)
@@ -26,20 +26,20 @@
         <rotors>
             <rotor>
-              <jointName>rotor_01_joint</jointName>
-              <linkName>rotor_01</linkName>
-              <spinDirection>ccw</spinDirection>
-              <timeConstantUp>${time_constant_up}</timeConstantUp>
-              <timeConstantDown>${time_constant_down}</timeConstantDown>
-              <minRotVelocity>${min_rot_velocity}</minRotVelocity>
-              <maxRotVelocity>${max_rot_velocity}</maxRotVelocity>
-              <thrustConstant>${motor_constant}</thrustConstant>
-              <momentConstant>${moment_constant}</momentConstant>
-              <rotorDragCoefficient>${rotor_drag_coefficient}</rotorDragCoefficient>
-              <rollingMomentCoefficient>${rolling_moment_coefficient}</rollingMomentCoefficient>
-              <rotorVelocitySlowdownSim>${rotor_velocity_slowdown_sim}</rotorVelocitySlowdownSim>
-            </rotor>
-            <rotor>
-              <jointName>rotor_02_joint</jointName>
-              <linkName>rotor_02</linkName>
+              <jointName>rotor_0_joint</jointName>
+              <linkName>rotor_0</linkName>
+              <spinDirection>ccw</spinDirection>
+              <timeConstantUp>${time_constant_up}</timeConstantUp>
+              <timeConstantDown>${time_constant_down}</timeConstantDown>
+              <minRotVelocity>${min_rot_velocity}</minRotVelocity>
+              <maxRotVelocity>${max_rot_velocity}</maxRotVelocity>
+              <thrustConstant>${motor_constant}</thrustConstant>
+              <momentConstant>${moment_constant}</momentConstant>
+              <rotorDragCoefficient>${rotor_drag_coefficient}</rotorDragCoefficient>
+              <rollingMomentCoefficient>${rolling_moment_coefficient}</rollingMomentCoefficient>
+              <rotorVelocitySlowdownSim>${rotor_velocity_slowdown_sim}</rotorVelocitySlowdownSim>
+            </rotor>
+            <rotor>
+              <jointName>rotor_4_joint</jointName>
+              <linkName>rotor_4</linkName>
               <spinDirection>cw</spinDirection>
               <timeConstantUp>${time_constant_up}</timeConstantUp>
@@ -54,20 +54,20 @@
             </rotor>
             <rotor>
-              <jointName>rotor_11_joint</jointName>
-              <linkName>rotor_11</linkName>
-              <spinDirection>ccw</spinDirection>
-              <timeConstantUp>${time_constant_up}</timeConstantUp>
-              <timeConstantDown>${time_constant_down}</timeConstantDown>
-              <minRotVelocity>${min_rot_velocity}</minRotVelocity>
-              <maxRotVelocity>${max_rot_velocity}</maxRotVelocity>
-              <thrustConstant>${motor_constant}</thrustConstant>
-              <momentConstant>${moment_constant}</momentConstant>
-              <rotorDragCoefficient>${rotor_drag_coefficient}</rotorDragCoefficient>
-              <rollingMomentCoefficient>${rolling_moment_coefficient}</rollingMomentCoefficient>
-              <rotorVelocitySlowdownSim>${rotor_velocity_slowdown_sim}</rotorVelocitySlowdownSim>
-            </rotor>
-            <rotor>
-              <jointName>rotor_12_joint</jointName>
-              <linkName>rotor_12</linkName>
+              <jointName>rotor_1_joint</jointName>
+              <linkName>rotor_1</linkName>
+              <spinDirection>ccw</spinDirection>
+              <timeConstantUp>${time_constant_up}</timeConstantUp>
+              <timeConstantDown>${time_constant_down}</timeConstantDown>
+              <minRotVelocity>${min_rot_velocity}</minRotVelocity>
+              <maxRotVelocity>${max_rot_velocity}</maxRotVelocity>
+              <thrustConstant>${motor_constant}</thrustConstant>
+              <momentConstant>${moment_constant}</momentConstant>
+              <rotorDragCoefficient>${rotor_drag_coefficient}</rotorDragCoefficient>
+              <rollingMomentCoefficient>${rolling_moment_coefficient}</rollingMomentCoefficient>
+              <rotorVelocitySlowdownSim>${rotor_velocity_slowdown_sim}</rotorVelocitySlowdownSim>
+            </rotor>
+            <rotor>
+              <jointName>rotor_5_joint</jointName>
+              <linkName>rotor_5</linkName>
               <spinDirection>cw</spinDirection>
               <timeConstantUp>${time_constant_up}</timeConstantUp>
@@ -82,6 +82,6 @@
             </rotor>
             <rotor>
-                <jointName>rotor_21_joint</jointName>
-                <linkName>rotor_21</linkName>
+                <jointName>rotor_2_joint</jointName>
+                <linkName>rotor_2</linkName>
                 <spinDirection>ccw</spinDirection>
                 <timeConstantUp>${time_constant_up}</timeConstantUp>
@@ -96,6 +96,6 @@
             </rotor>
             <rotor>
-                <jointName>rotor_22_joint</jointName>
-                <linkName>rotor_22</linkName>
+                <jointName>rotor_6_joint</jointName>
+                <linkName>rotor_6</linkName>
                 <spinDirection>cw</spinDirection>
                 <timeConstantUp>${time_constant_up}</timeConstantUp>
@@ -110,6 +110,6 @@
             </rotor>
             <rotor>
-                <jointName>rotor_31_joint</jointName>
-                <linkName>rotor_31</linkName>
+                <jointName>rotor_3_joint</jointName>
+                <linkName>rotor_3</linkName>
                 <spinDirection>ccw</spinDirection>
                 <timeConstantUp>${time_constant_up}</timeConstantUp>
@@ -124,6 +124,6 @@
             </rotor>
             <rotor>
-                <jointName>rotor_32_joint</jointName>
-                <linkName>rotor_32</linkName>
+                <jointName>rotor_7_joint</jointName>
+                <linkName>rotor_7</linkName>
                 <spinDirection>cw</spinDirection>
                 <timeConstantUp>${time_constant_up}</timeConstantUp>

File: rotors_description/urdf/omav_snippets.xacro (robot description, xacro)
@@ -280,11 +280,11 @@
     </gazebo>
     <!-- Upper Rotor -->
-    <joint name="rotor_${motor_number}1_joint" type="continuous">
+    <joint name="rotor_${motor_number}_joint" type="continuous">
       <origin xyz="0 0 ${rotor_offset_top}" rpy="0 0 0" />
       <axis xyz="0 0 1" />
       <parent link="${namespace}/tilt_unit_${motor_number}" />
-      <child link="rotor_${motor_number}1" />
-    </joint>
-    <link name="rotor_${motor_number}1">
+      <child link="rotor_${motor_number}" />
+    </joint>
+    <link name="rotor_${motor_number}">
       <inertial>
         <mass value="${mass_rotor}" /> <!-- [kg] -->
@@ -303,15 +303,15 @@
       </collision>
     </link>
-    <gazebo reference="rotor_${motor_number}1">
+    <gazebo reference="rotor_${motor_number}">
       <material>Gazebo/${color}</material>
     </gazebo>
     <!-- Lower Rotor -->
-    <joint name="rotor_${motor_number}2_joint" type="continuous">
+    <joint name="rotor_${motor_number+4}_joint" type="continuous">
       <origin xyz="0 0 ${-rotor_offset_top}" rpy="0 0 0" />
       <axis xyz="0 0 1" />
       <parent link="${namespace}/tilt_unit_${motor_number}" />
-      <child link="rotor_${motor_number}2" />
-    </joint>
-    <link name="rotor_${motor_number}2">
+      <child link="rotor_${motor_number+4}" />
+    </joint>
+    <link name="rotor_${motor_number+4}">
       <inertial>
         <mass value="${mass_rotor}" /> <!-- [kg] -->
@@ -330,5 +330,5 @@
       </collision>
     </link>
-    <gazebo reference="rotor_${motor_number}2">
+    <gazebo reference="rotor_${motor_number+4}">
       <material>Gazebo/${color}</material>
     </gazebo>

Commit message: Minimal double rotor group + griffin.

File: rotors_description/urdf/griffin.xacro (robot description, xacro)
@@ -45,4 +45,5 @@
   <xacro:property name="cos60" value="0.5"/>
   <xacro:property name="sin60" value="0.866025403784"/>
+  <xacro:property name="num_rotor_groups" value="4"/>
   <!-- Property Blocks -->
   <xacro:property name="body_inertia">
@@ -88,4 +89,5 @@
           rotor_offset_top="${rotor_offset_top}"
           motor_number="0"
+          lower_start_index="${num_rotor_groups}"
           mesh="propeller"
           mesh_tilt_unit="${mesh_file_tilt_unit}"
@@ -104,4 +106,5 @@
           rotor_offset_top="${rotor_offset_top}"
           motor_number="1"
+          lower_start_index="${num_rotor_groups}"
           mesh="propeller"
           mesh_tilt_unit="${mesh_file_tilt_unit}"
@@ -120,4 +123,5 @@
           rotor_offset_top="${rotor_offset_top}"
           motor_number="2"
+          lower_start_index="${num_rotor_groups}"
           mesh="propeller"
           mesh_tilt_unit="${mesh_file_tilt_unit}"
@@ -136,4 +140,5 @@
           rotor_offset_top="${rotor_offset_top}"
           motor_number="3"
+          lower_start_index="${num_rotor_groups}"
           mesh="propeller"
           mesh_tilt_unit="${mesh_file_tilt_unit}"

File: rotors_description/urdf/omav_snippets.xacro (robot description, xacro)
@@ -391,3 +391,91 @@
     </gazebo>
   </xacro:macro>
+  <!-- Tilting double rotor unit link and joint. -->
+  <xacro:macro name="double_tilt_unit_minimal"
+    params="robot_namespace direction_upper direction_lower parent mass_rotor mass_tilt_unit rotor_offset_top motor_number lower_start_index color mesh mesh_tilt_unit *origin *inertia">
+    <!-- Rotor tilt_unit -->
+    <joint name="${robot_namespace}/tilt_unit_${motor_number}_revolutejoint" type="continuous">
+      <xacro:insert_block name="origin" />
+      <axis xyz="1 0 0" />
+      <parent link="${parent}" />
+      <child link="${namespace}/tilt_unit_${motor_number}" />
+    </joint>
+    <gazebo reference="${robot_namespace}/tilt_unit_${motor_number}_revolutejoint">
+      <provideFeedback>true</provideFeedback>
+    </gazebo>
+    <link name="${namespace}/tilt_unit_${motor_number}">
+      <inertial>
+        <mass value="${mass_tilt_unit}" /> <!-- [kg] -->
+        <xacro:insert_block name="tilt_unit_inertia" />
+      </inertial>
+      <visual>
+        <geometry>
+            <mesh filename="${mesh_tilt_unit}"
+              scale="1 1 1" />
+        </geometry>
+      </visual>
+      <collision>
+        <geometry>
+          <box size="0.005 0.005 0.005"  /> <!-- [m] -->
+        </geometry>
+      </collision>
+    </link>
+    <gazebo reference="${namespace}/tilt_unit_${motor_number}">
+      <material>Gazebo/White</material>
+    </gazebo>
+    <!-- Upper Rotor -->
+    <joint name="rotor_${motor_number}_joint" type="continuous">
+      <origin xyz="0 0 ${rotor_offset_top}" rpy="0 0 0" />
+      <axis xyz="0 0 1" />
+      <parent link="${namespace}/tilt_unit_${motor_number}" />
+      <child link="rotor_${motor_number}" />
+    </joint>
+    <link name="rotor_${motor_number}">
+      <inertial>
+        <mass value="${mass_rotor}" /> <!-- [kg] -->
+        <xacro:insert_block name="inertia" />
+      </inertial>
+      <visual>
+        <geometry>
+          <mesh filename="package://rotors_description/meshes/${mesh}_${direction_upper}.dae"
+            scale="${radius_rotor} ${radius_rotor} ${radius_rotor}" />
+        </geometry>
+      </visual>
+      <collision>
+        <geometry>
+          <cylinder length="0.005" radius="${radius_rotor}" /> <!-- [m] -->
+        </geometry>
+      </collision>
+    </link>
+    <gazebo reference="rotor_${motor_number}">
+      <material>Gazebo/${color}</material>
+    </gazebo>
+    <!-- Lower Rotor -->
+    <joint name="rotor_${motor_number+lower_start_index}_joint" type="continuous">
+      <origin xyz="0 0 ${-rotor_offset_top}" rpy="0 0 0" />
+      <axis xyz="0 0 1" />
+      <parent link="${namespace}/tilt_unit_${motor_number}" />
+      <child link="rotor_${motor_number+lower_start_index}" />
+    </joint>
+    <link name="rotor_${motor_number+lower_start_index}">
+      <inertial>
+        <mass value="${mass_rotor}" /> <!-- [kg] -->
+        <xacro:insert_block name="inertia" />
+      </inertial>
+      <visual>
+        <geometry>
+          <mesh filename="package://rotors_description/meshes/${mesh}_${direction_lower}.dae"
+            scale="${radius_rotor} ${radius_rotor} ${radius_rotor}" />
+        </geometry>
+      </visual>
+      <collision>
+        <geometry>
+          <cylinder length="0.005" radius="${radius_rotor}" /> <!-- [m] -->
+        </geometry>
+      </collision>
+    </link>
+    <gazebo reference="rotor_${motor_number+lower_start_index}">
+      <material>Gazebo/${color}</material>
+    </gazebo>
+  </xacro:macro>
 </robot>
