Commit message: fixes

File: rotors_description/urdf/griffin.xacro (robot description, xacro)
@@ -25,19 +25,19 @@
   <xacro:property name="use_mesh_file_rotor_unit" value="true"/>
   <xacro:property name="mesh_file_core" value="package://rotors_description/meshes/omav/griffin_base.stl"/>
-  <xacro:property name="mesh_file_core_collision" value="package://rotors_description/meshes/omav/griffin_base.stl"/>
+  <xacro:property name="mesh_file_core_collision" value="package://rotors_description/meshes/omav/griffin_base.stl"/> //TODO what is this for
   <xacro:property name="mesh_file_tilt_unit" value="package://rotors_description/meshes/omav/griffin_tilt_unit.stl"/>
-  <xacro:property name="mass_core" value="6.57"/>    <!-- [kg] -->
+  <xacro:property name="mass_core" value="6.57"/>    <!-- [kg] --> //TODO evtl kleiner
   <xacro:property name="mass_tilt_unit" value="0.33"/>    <!-- [kg] -->
-  <xacro:property name="body_width" value="0.22"/>    <!-- [m] TODO -->
-  <xacro:property name="body_height" value="0.666"/>    <!-- [m] TODO -->
+  <xacro:property name="body_width" value="0.8"/>    <!-- [m]  -->
+  <xacro:property name="body_height" value="1.2"/>    <!-- [m]  -->
   <xacro:property name="mass_rotor" value="0.045"/>    <!-- [kg] -->
-  <xacro:property name="arm_length_front" value="0.35"/> <!-- [m] -->
-  <xacro:property name="arm_length_back" value="0.595"/> <!-- [m] -->
+  <xacro:property name="arm_length_front" value="0.4"/> <!-- [m] -->
+  <xacro:property name="arm_length_back" value="0.6"/> <!-- [m] -->
   <xacro:property name="rotor_offset_top" value="0.0445"/>    <!-- [m] -->
-  <xacro:property name="radius_rotor" value="${0.406/2}"/>    <!-- 12 in [m] -->
+  <xacro:property name="radius_rotor" value="${0.406/2}"/>    <!-- 16 in props/2 [m] -->
   <xacro:property name="mass_tilt_unit_back" value="0.32"/> <!-- [kg] -->
   <xacro:property name="tilt_unit_parent" value="${namespace}/base_link_inertia"/>    <!-- 12 in [m] -->
   <xacro:property name="body_origin">
-    <origin xyz="0 0 0" rpy="${mounting_roll} 0 0" />
+    <origin xyz="0 0 0" rpy="0 0 0" />
   </xacro:property>
   <xacro:property name="sin30" value="0.5"/>
@@ -126,5 +126,5 @@
           mesh="propeller"
           mesh_tilt_unit="${mesh_file_tilt_unit}"
-          color="Orange">
+          color="Black">
     <origin xyz="-${arm_length_front*cos30} -${arm_length_front*sin30} 0" rpy="0 0 -2.61799387799"/>
     <xacro:insert_block name="rotor_inertia" />
@@ -143,5 +143,5 @@
           mesh="propeller"
           mesh_tilt_unit="${mesh_file_tilt_unit}"
-          color="DarkGrey">
+          color="Orange">
     <origin xyz="0 0 ${arm_length_back}" rpy="0 -1.57079632679 0"/>
     <xacro:insert_block name="rotor_inertia" />

File: rotors_description/urdf/griffin_actuators.xacro (robot description, xacro)
@@ -7,5 +7,5 @@
   <xacro:property name="time_constant_down" value="0.025"/>    <!-- [s] -->
   <xacro:property name="min_rot_velocity" value="100"/>
-  <xacro:property name="max_rot_velocity" value="1700"/>    <!-- [rad/s] --> <!-- Velocity to produce 1 kg thrust -->
+  <xacro:property name="max_rot_velocity" value="7000"/>    <!-- [rad/s] --> <!-- Velocity to produce 1 kg thrust -->
   <xacro:property name="rotor_drag_coefficient" value="${8.06428e-05}"/>
   <xacro:property name="rolling_moment_coefficient" value="0.000001"/>

File: rotors_description/urdf/griffin_base.xacro (robot description, xacro)
@@ -2,16 +2,6 @@
 <robot name="$(arg mav_name)" xmlns:xacro="http://ros.org/wiki/xacro">
     <xacro:include filename="$(find rotors_description)/urdf/component_snippets.xacro"/>
-    <xacro:property name="mounting_roll" value="$(arg model_roll)" />
     <!-- Instantiate OMAV "mechanics". -->
     <xacro:include filename="$(find rotors_description)/urdf/griffin.xacro"/>
-    <!-- Add manipulator. -->
-    <xacro:if value="$(arg add_manipulator)">
-        <xacro:property name="robot_name" value="delta" />
-        <xacro:property name="delta_namespace" value="delta" />
-        <xacro:property name="mounting_link" value="$(arg mav_name)/base_link" />
-        <xacro:property name="height_offset" value="0.073" />
-        <xacro:include filename="$(find rotors_description)/urdf/delta_manipulator.xacro" />
-        <xacro:include filename="$(find rotors_description)/urdf/delta_actuators.xacro" />
-    </xacro:if>
     <xacro:include filename="$(find rotors_description)/urdf/griffin_actuators.xacro" />
     <!-- Mount an ADIS16448 IMU. -->
@@ -48,13 +38,4 @@
                 wait_to_record_bag="$(arg wait_to_record_bag)"/>
     </xacro:if>
-    <xacro:if value="$(arg add_rgbd_sensor)">
-        <!-- Add a RGB-D sensor -->
-        <xacro:include filename="$(find rotors_description)/urdf/pmd_monstar.xacro"/>
-        <joint name="$(arg mav_name)/tof_cam_optical_frame" type="fixed">
-            <origin xyz="0.09 0.0 0.15" rpy="-1.309 0 -1.571"/>
-            <parent link="$(arg mav_name)/base_link_inertia" />
-            <child link="rgbd_camera/base_link" />
-        </joint>
-    </xacro:if>
     <!-- Add odometry. -->
     <xacro:include filename="$(find rotors_description)/urdf/odometry_sensor_smooth.xacro"/>

Commit message: für phillippe

File: rotors_description/urdf/griffin.xacro (robot description, xacro)
@@ -39,5 +39,5 @@
   <xacro:property name="tilt_unit_parent" value="${namespace}/base_link_inertia"/>    <!-- 12 in [m] -->
   <xacro:property name="body_origin">
-    <origin xyz="0 0 0" rpy="0 0 0" />
+    <origin xyz="0 0 0.121" rpy="0 0 0" />
   </xacro:property>
   <xacro:property name="sin30" value="0.5"/>
@@ -54,5 +54,5 @@
   <xacro:property name="body_inertia_origin">
     <!-- <origin xyz="0.03 0 0.01" /> -->
-    <origin xyz="-0.0024 -0.0035 0.121" /> <!-- [m] -->
+    <origin xyz="0 0 0" /> <!-- [m] -->
   </xacro:property>
   <!-- Rotor unit inertia without the propellor. -->
@@ -110,5 +110,5 @@
           mesh_tilt_unit="${mesh_file_tilt_unit}"
           color="Black">
-    <origin xyz="${arm_length_front*cos30} -${arm_length_front*sin30} 0" rpy="0 0 -0.52359877559"/>
+    <origin xyz="-${arm_length_front*cos30} -${arm_length_front*sin30} 0" rpy="0 0 -2.61799387799"/>
     <xacro:insert_block name="rotor_inertia" />
   </xacro:double_tilt_unit_minimal>
@@ -127,5 +127,5 @@
           mesh_tilt_unit="${mesh_file_tilt_unit}"
           color="Black">
-    <origin xyz="-${arm_length_front*cos30} -${arm_length_front*sin30} 0" rpy="0 0 -2.61799387799"/>
+    <origin xyz="${arm_length_front*cos30} -${arm_length_front*sin30} 0" rpy="0 0 -0.52359877559"/>
     <xacro:insert_block name="rotor_inertia" />
   </xacro:double_tilt_unit_minimal>

File: rotors_description/urdf/griffin_base.xacro (robot description, xacro)
@@ -23,5 +23,5 @@
             measurement_divisor="2">
         <inertia ixx="0.00001" ixy="0.0" ixz="0.0" iyy="0.00001" iyz="0.0" izz="0.00001" />
-        <origin xyz="0 0 0" rpy="0 0 0" />
+        <origin xyz="0 0 0.121" rpy="0 0 0" />
     </xacro:imu_plugin_macro>
     <xacro:if value="$(arg enable_ground_truth)">
